Commit message: plugin + visu dans un script

File: urdf/my_turtlebot3_ultimate.urdf (robot description, URDF)
Before this commit: robot turtlebot3_burger_ultimate, 15 links, 14 joints
Joints:
- joint joint_oak_d_pro_camera: origin xyz=0.065 0.0 0.11 rpy=1.57 0.0 1.57 -> xyz=0.09 0.0 0.145 rpy=1.57 0.0 1.57

Commit message: modif pour que la camera regarde bien devant

File: urdf/my_turtlebot3_ultimate.urdf (robot description, URDF)
Before this commit: robot turtlebot3_burger_ultimate, 15 links, 14 joints
Joints:
- joint joint_oak_d_pro_camera: origin xyz=0.09 0.0 0.145 rpy=1.57 0.0 1.57 -> xyz=0.09 0.0 0.145 rpy=0 0 0
- joint joint_oak_d_pro_color_optical_frame: origin xyz=0.0 0.0 0.0 rpy=-1.5708 0.0 -1.5708 -> xyz=0 0 0 rpy=0 0 0
- joint oak_d_pro_depth_optical_frame: origin xyz=0.0 0.0 0.0 rpy=-1.5708 0.0 -1.5708 -> xyz=0 0 0 rpy=0 0 0
