Commit message: Added node for gripper
-Add CatchNode for gripper control and update URDF joint naming

File: urdf/turtlebot3_ultimate.urdf (robot description, URDF)
Before this commit: robot turtlebot3_burger_ultimate, 15 links, 14 joints
Joints:
- joint gripper_right_joint: mimic (none) -> joint=gripper_left_joint multiplier=-1 offset=0
