Commit message: omg le robot avec la pince roule nikel

File: urdf/my_turtlebot.urdf (robot description, URDF)
Before this commit: robot turtlebot3_waffle, 16 links, 15 joints
Links:
- removed link ${namespace}caster_back_left_link
- removed link ${namespace}caster_back_right_link
- added link ${namespace}caster_back_link, mass 0.005; collision sphere radius=0.015
- added link ${namespace}caster_front_link, mass 0.005; collision sphere radius=0.015
- link ${namespace}base_link: mass 1.3729096e+00 -> 0.82573504e+00; geometry collision box size=0.140 0.140 0.143; visual mesh filename=package://turtlebot3_description/meshes/bases/burger_base.s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 scale=0.001 0.001 0.001
Joints:
- removed joint ${namespace}caster_back_left_joint
- removed joint ${namespace}caster_back_right_joint
- added joint ${namespace}caster_back_joint: type fixed, parent ${namespace}base_link, child ${namespace}caster_back_link, origin xyz=-0.081 0 -0.004 rpy=-1.57 0 0
- added joint ${namespace}caster_front_joint: type fixed, parent ${namespace}base_link, child ${namespace}caster_front_link, origin xyz=0.081 0 0.010 rpy=-1.57 0 0
- joint ${namespace}imu_joint: origin xyz=0.0 0 0.068 rpy=0 0 0 -> xyz=-0.032 0 0.068 rpy=0 0 0
- joint ${namespace}scan_joint: origin xyz=-0.064 0 0.122 rpy=0 0 0 -> xyz=-0.032 0 0.172 rpy=0 0 0
- joint ${namespace}wheel_left_joint: origin xyz=0.0 0.144 0.023 rpy=-1.57 0 0 -> xyz=0.0 0.08 0.023 rpy=-1.57 0 0
- joint ${namespace}wheel_right_joint: origin xyz=0.0 -0.144 0.023 rpy=-1.57 0 0 -> xyz=0.0 -0.08 0.023 rpy=-1.57 0 0
- joint oakd_joint: origin xyz=0.064 0 0.094 rpy=0 0.26 0 -> xyz=0.04 0 0.13 rpy=0 0.15 0

Commit message: correction cam + test cible de trajet

File: urdf/my_turtlebot.urdf (robot description, URDF)
Before this commit: robot turtlebot3_burger, 16 links, 15 joints
Links:
- removed link ${namespace}base_footprint
- removed link ${namespace}base_link
- removed link ${namespace}base_scan
- removed link ${namespace}caster_back_link
- removed link ${namespace}caster_front_link
- removed link ${namespace}imu_link
- removed link ${namespace}wheel_left_link
- removed link ${namespace}wheel_right_link
- removed link oakd_imu_frame
- removed link oakd_left_frame
- removed link oakd_left_optical_frame
- removed link oakd_link
- removed link oakd_rgb_frame
- removed link oakd_rgb_optical_frame
- removed link oakd_right_frame
- removed link oakd_right_optical_frame
- added link base_footprint
- added link base_gripper, mass 0.06; collision box size=0.03 0.055 0.06; visual mesh filename=package://tb3_autonomy/meshes/gripper_base.stl scale=0.001 0.001 0.001
- added link base_link, mass 0.82573504; collision box size=0.140 0.140 0.143; visual mesh filename=package://turtlebot3_description/meshes/bases/burger_base.s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 scale=0.001 0.001 0.001
- added link base_scan, mass 0.114; collision cylinder length=0.0315 radius=0.055; visual mesh filename=package://turtlebot3_description/meshes/sensors/lds.stl scale=0.001 0.001 0.001
- added link caster_back_link, mass 0.005; collision box size=0.030 0.009 0.020
- added link counterweight_link, mass 0.5; visual box size=0.05 0.1 0.05
- added link imu_link
- added link left_gripper, mass 0.120; collision box size=0.02 0.02 0.041; visual mesh filename=package://tb3_autonomy/meshes/gripper_left.stl scale=0.001 0.001 0.001
- added link oak_d_pro_camera, mass 0.091; collision box size=0.1 0.03 0.02; visual mesh filename=package://tb3_autonomy/meshes/OAK-D-PRO.stl scale=1.0 1.0 1.0
- added link oak_d_pro_color_optical_frame
- added link oak_d_pro_depth_optical_frame
- added link right_gripper, mass 0.120; collision box size=0.02 0.02 0.041; visual mesh filename=package://tb3_autonomy/meshes/gripper_right.stl scale=0.001 0.001 0.001
- added link tilt_gripper, mass 0.060; collision box size=0.055 0.075 0.06; visual mesh filename=package://tb3_autonomy/meshes/gripper_tilt.stl scale=0.001 0.001 0.001
- added link wheel_left_link, mass 0.02849894; collision cylinder length=0.018 radius=0.033; visual mesh filename=package://turtlebot3_description/meshes/wheels/left_tire.stl scale=0.001 0.001 0.001
- added link wheel_right_link, mass 0.02849894; collision cylinder length=0.018 radius=0.033; visual mesh filename=package://turtlebot3_description/meshes/wheels/right_tire.s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 scale=0.001 0.001 0.001
Joints:
- removed joint ${namespace}base_joint
- removed joint ${namespace}caster_back_joint
- removed joint ${namespace}caster_front_joint
- removed joint ${namespace}imu_joint
- removed joint ${namespace}scan_joint
- removed joint ${namespace}wheel_left_joint
- removed joint ${namespace}wheel_right_joint
- removed joint oakd_imu_joint
- removed joint oakd_joint
- removed joint oakd_left_joint
- removed joint oakd_left_optical_joint
- removed joint oakd_rgb_joint
- removed joint oakd_rgb_optical_joint
- removed joint oakd_right_joint
- removed joint oakd_right_optical_joint
- added joint base_joint: type fixed, parent base_footprint, child base_link, origin xyz=0.0 0.0 0.010 rpy=0 0 0
- added joint caster_back_joint: type fixed, parent base_link, child caster_back_link, origin xyz=-0.081 0 -0.004 rpy=-1.57 0 0
- added joint counterweight_joint: type fixed, parent base_link, child counterweight_link, origin xyz=-0.15 0 0.05 rpy=0 0 0
- added joint gripper_base_joint: type fixed, parent base_link, child base_gripper, origin xyz=0.052 0.0025 0.04 rpy=0 0 0
- added joint gripper_left_joint: type revolute, parent tilt_gripper, child left_gripper, origin xyz=0.05 0.016 0.018 rpy=0 0 0, axis 0 0 1, limit lower=0 upper=1.0 effort=1000.0 velocity=0.5
- added joint gripper_right_joint: type revolute, parent tilt_gripper, child right_gripper, origin xyz=0.05 -0.016 0.018 rpy=0 0 0, axis 0 0 1, limit lower=-1.0 upper=0 effort=1000.0 velocity=0.5
- added joint gripper_tilt_joint: type revolute, parent base_gripper, child tilt_gripper, origin xyz=0 0.002 0 rpy=0 0 0, axis 0 1 0, limit lower=-0.3 upper=0 effort=1000.0 velocity=0.5
- added joint imu_joint: type fixed, parent base_link, child imu_link, origin xyz=-0.032 0 0.068 rpy=0 0 0
- added joint joint_oak_d_pro_camera: type fixed, parent base_link, child oak_d_pro_camera, origin xyz=0.09 0.0 0.145 rpy=0 0 0
- added joint joint_oak_d_pro_color_optical_frame: type fixed, parent oak_d_pro_camera, child oak_d_pro_color_optical_frame, origin xyz=0 0 0 rpy=0 0 0
- added joint oak_d_pro_depth_optical_frame: type fixed, parent oak_d_pro_camera, child oak_d_pro_depth_optical_frame, origin xyz=0 0 0 rpy=0 0 0
- added joint scan_joint: type fixed, parent base_link, child base_scan, origin xyz=-0.032 0 0.172 rpy=0 0 0
- added joint wheel_left_joint: type continuous, parent base_link, child wheel_left_link, origin xyz=0.0 0.08 0.023 rpy=-1.57 0 0, axis 0 0 1
- added joint wheel_right_joint: type continuous, parent base_link, child wheel_right_link, origin xyz=0.0 -0.080 0.023 rpy=-1.57 0 0, axis 0 0 1

File: urdf/my_turtlebotold.urdf (robot description, URDF)
Before this commit: robot turtlebot3_waffle, 16 links, 15 joints
Links:
- removed link ${namespace}base_footprint
- removed link ${namespace}base_link
- removed link ${namespace}base_scan
- removed link ${namespace}caster_back_left_link
- removed link ${namespace}caster_back_right_link
- removed link ${namespace}imu_link
- removed link ${namespace}wheel_left_link
- removed link ${namespace}wheel_right_link
- removed link oakd_imu_frame
- removed link oakd_left_frame
- removed link oakd_left_optical_frame
- removed link oakd_link
- removed link oakd_rgb_frame
- removed link oakd_rgb_optical_frame
- removed link oakd_right_frame
- removed link oakd_right_optical_frame
- added link base_footprint
- added link base_gripper, mass 0.06; collision box size=0.03 0.055 0.06; visual mesh filename=package://tb3_autonomy/meshes/gripper_base.stl scale=0.001 0.001 0.001
- added link base_link, mass 0.82573504; collision box size=0.140 0.140 0.143; visual mesh filename=package://turtlebot3_description/meshes/bases/burger_base.s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 scale=0.001 0.001 0.001
- added link base_scan, mass 0.114; collision cylinder length=0.0315 radius=0.055; visual mesh filename=package://turtlebot3_description/meshes/sensors/lds.stl scale=0.001 0.001 0.001
- added link caster_back_link, mass 0.005; collision box size=0.030 0.009 0.020
- added link counterweight_link, mass 0.5; visual box size=0.05 0.1 0.05
- added link imu_link
- added link left_gripper, mass 0.120; collision box size=0.02 0.02 0.041; visual mesh filename=package://tb3_autonomy/meshes/gripper_left.stl scale=0.001 0.001 0.001
- added link oak_d_pro_camera, mass 0.091; collision box size=0.1 0.03 0.02; visual mesh filename=package://tb3_autonomy/meshes/OAK-D-PRO.stl scale=1.0 1.0 1.0
- added link oak_d_pro_color_optical_frame
- added link oak_d_pro_depth_optical_frame
- added link right_gripper, mass 0.120; collision box size=0.02 0.02 0.041; visual mesh filename=package://tb3_autonomy/meshes/gripper_right.stl scale=0.001 0.001 0.001
- added link tilt_gripper, mass 0.060; collision box size=0.055 0.075 0.06; visual mesh filename=package://tb3_autonomy/meshes/gripper_tilt.stl scale=0.001 0.001 0.001
- added link wheel_left_link, mass 0.02849894; collision cylinder length=0.018 radius=0.033; visual mesh filename=package://turtlebot3_description/meshes/wheels/left_tire.stl scale=0.001 0.001 0.001
- added link wheel_right_link, mass 0.02849894; collision cylinder length=0.018 radius=0.033; visual mesh filename=package://turtlebot3_description/meshes/wheels/right_tire.s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 scale=0.001 0.001 0.001
Joints:
- removed joint ${namespace}base_joint
- removed joint ${namespace}caster_back_left_joint
- removed joint ${namespace}caster_back_right_joint
- removed joint ${namespace}imu_joint
- removed joint ${namespace}scan_joint
- removed joint ${namespace}wheel_left_joint
- removed joint ${namespace}wheel_right_joint
- removed joint oakd_imu_joint
- removed joint oakd_joint
- removed joint oakd_left_joint
- removed joint oakd_left_optical_joint
- removed joint oakd_rgb_joint
- removed joint oakd_rgb_optical_joint
- removed joint oakd_right_joint
- removed joint oakd_right_optical_joint
- added joint base_joint: type fixed, parent base_footprint, child base_link, origin xyz=0.0 0.0 0.010 rpy=0 0 0
- added joint caster_back_joint: type fixed, parent base_link, child caster_back_link, origin xyz=-0.081 0 -0.004 rpy=-1.57 0 0
- added joint counterweight_joint: type fixed, parent base_link, child counterweight_link, origin xyz=-0.15 0 0.05 rpy=0 0 0
- added joint gripper_base_joint: type fixed, parent base_link, child base_gripper, origin xyz=0.052 0.0025 0.04 rpy=0 0 0
- added joint gripper_left_joint: type revolute, parent tilt_gripper, child left_gripper, origin xyz=0.05 0.016 0.018 rpy=0 0 0, axis 0 0 1, limit lower=0 upper=1.0 effort=1000.0 velocity=0.5
- added joint gripper_right_joint: type revolute, parent tilt_gripper, child right_gripper, origin xyz=0.05 -0.016 0.018 rpy=0 0 0, axis 0 0 1, limit lower=-1.0 upper=0 effort=1000.0 velocity=0.5
- added joint gripper_tilt_joint: type revolute, parent base_gripper, child tilt_gripper, origin xyz=0 0.002 0 rpy=0 0 0, axis 0 1 0, limit lower=-0.3 upper=0 effort=1000.0 velocity=0.5
- added joint imu_joint: type fixed, parent base_link, child imu_link, origin xyz=-0.032 0 0.068 rpy=0 0 0
- added joint joint_oak_d_pro_camera: type fixed, parent base_link, child oak_d_pro_camera, origin xyz=0.09 0.0 0.145 rpy=0 0 0
- added joint joint_oak_d_pro_color_optical_frame: type fixed, parent oak_d_pro_camera, child oak_d_pro_color_optical_frame, origin xyz=0 0 0 rpy=0 0 0
- added joint oak_d_pro_depth_optical_frame: type fixed, parent oak_d_pro_camera, child oak_d_pro_depth_optical_frame, origin xyz=0 0 0 rpy=0 0 0
- added joint scan_joint: type fixed, parent base_link, child base_scan, origin xyz=-0.032 0 0.172 rpy=0 0 0
- added joint wheel_left_joint: type continuous, parent base_link, child wheel_left_link, origin xyz=0.0 0.08 0.023 rpy=-1.57 0 0, axis 0 0 1
- added joint wheel_right_joint: type continuous, parent base_link, child wheel_right_link, origin xyz=0.0 -0.080 0.023 rpy=-1.57 0 0, axis 0 0 1
