Commit message: affiche correct mais prb texture

File: urdf/turtlebot3_burger_gripper.urdf (robot description, URDF)
Before this commit: robot turtlebot3_burger, 17 links, 16 joints
Links:
- link base_gripper: geometry collision box size=0.055 0.055 0.06; visual mesh filename=package://tb3_autonomy/meshes/actuators/gripper/gripper_bas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 scale=0.001 0.001 0.001
- link base_link: geometry collision box size=0.140 0.140 0.143; visual mesh filename=package://tb3_autonomy/meshes/bases/burger_base.stl scale=0.001 0.001 0.001
- link base_scan: geometry collision cylinder length=0.0315 radius=0.055; visual mesh filename=package://tb3_autonomy/meshes/sensors/lds.stl scale=0.001 0.001 0.001
- link left_gripper: geometry collision box size=0.02 0.02 0.041; visual mesh filename=package://tb3_autonomy/meshes/actuators/gripper/gripper_lef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 scale=0.001 0.001 0.001
- link oak_d_pro_camera: geometry collision box size=0.1 0.03 0.02; visual mesh filename=package://tb3_autonomy/meshes/sensors/OAK-D-PRO.stl scale=1.0 1.0 1.0
- link right_gripper: geometry collision box size=0.02 0.02 0.041; visual mesh filename=package://tb3_autonomy/meshes/actuators/gripper/gripper_rig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 scale=0.001 0.001 0.001
- link support_cameras_a_link: geometry collision box size=0.09 0.03 0.015; visual mesh filename=package://tb3_autonomy/meshes/sensors/support_cameras_part_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 scale=0.001 0.001 0.001
- link support_cameras_b_link: geometry collision box size=0.09 0.025 0.015; visual mesh filename=package://tb3_autonomy/meshes/sensors/support_cameras_part_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 scale=0.001 0.001 0.001
- link tilt_gripper: geometry collision box size=0.055 0.075 0.06; visual mesh filename=package://tb3_autonomy/meshes/actuators/gripper/gripper_til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 scale=0.001 0.001 0.001
- link wheel_left_link: geometry collision cylinder length=0.018 radius=0.033; visual mesh filename=package://tb3_autonomy/meshes/wheels/left_tire.stl scale=0.001 0.001 0.001
- link wheel_right_link: geometry collision cylinder length=0.018 radius=0.033; visual mesh filename=package://tb3_autonomy/meshes/wheels/right_tire.stl scale=0.001 0.001 0.001
