Commit message: FIX PINCE + clean + xacro + CA PINCE!

File: urdf/turtlebot3_burger_gripper.urdf.xacro (robot description, xacro)
@@ -1,9 +1,5 @@
-<?xml version="1.0" ?>
-<!-- =================================================================================== -->
-<!-- |    This document was autogenerated by xacro from turtlebot3_burger.urdf         | -->
-<!-- |    EDITING THIS FILE BY HAND IS NOT RECOMMENDED                                 | -->
-<!-- =================================================================================== -->
-<robot name="turtlebot3_burger">
-  <!-- <xacro:include filename="$(find tb3_autonomy)/urdf/common_properties.urdf"/> -->
+<?xml version="1.0"?>
+<robot name="turtlebot3_burger_gripper" xmlns:xacro="http://www.ros.org/wiki/xacro">
+  <xacro:arg name="controllers_file" default=""/>
   <!-- Init colour -->
   <material name="black">
@@ -339,5 +335,5 @@
     <parent link="oak_d_pro_camera"/>
     <child link="oak_d_pro_color_optical_frame"/>
-    <origin xyz="0.0 0.0 0.0" rpy="0 0 0"/>
+    <origin xyz="0 0 0" rpy="-1.5708 0 -1.5708"/>
   </joint>
   <link name="oak_d_pro_depth_optical_frame"/>
@@ -360,4 +356,11 @@
     <child link="counterweight"/>
     <origin xyz="-0.12 0.0 0.0" rpy="0 0 0"/>
+  </joint>
+  <link name="oak_d_pro_camera_gz"/>
+  <joint name="joint_oak_d_pro_camera_gz" type="fixed">
+    <parent link="oak_d_pro_camera"/>
+    <child link="oak_d_pro_camera_gz"/>
+    <!-- origin xyz="0 0 0" rpy="0 0 -1.5708"/>-->
+    <origin xyz="0 0 0" rpy="0 -1.57 -1.5708"/>
   </joint>
   <gazebo reference="imu_link">
@@ -389,41 +392,40 @@
   <!-- LIDAR 2D (Gazebo Classic = ray/gpu_ray + <ray> ... ) -->
   <gazebo reference="base_scan">
-    <sensor name="hls_lfcd_lds" type="gpu_ray">
-      <always_on>true</always_on>
-      <visualize>true</visualize>
-      <update_rate>15</update_rate>
-      <ray>
-        <scan>
-          <horizontal>
-            <samples>360</samples>
-            <resolution>1</resolution>
-            <min_angle>0.0</min_angle>
-            <max_angle>6.28</max_angle>
-          </horizontal>
-        </scan>
-        <range>
-          <min>0.12</min>
-          <max>3.5</max>
-          <resolution>0.015</resolution>
-        </range>
-        <noise type="gaussian">
-          <mean>0.0</mean>
-          <stddev>0.01</stddev>
-        </noise>
-      </ray>
-      <plugin name="tb3_laser_ros" filename="libgazebo_ros_ray_sensor.so">
-        <ros>
-          <namespace>/</namespace>
-          <remapping>~/out:=scan</remapping>
-        </ros>
-        <output_type>sensor_msgs/LaserScan</output_type>
-        <frame_name>base_scan</frame_name>
-      </plugin>
-    </sensor>
-  </gazebo>
+      <sensor name="hls_lfcd_lds" type="ray">
+        <always_on>true</always_on>
+        <visualize>false</visualize> <pose>0 0 0.01 0 0 0</pose> <update_rate>5</update_rate>
+        <ray>
+          <scan>
+            <horizontal>
+              <samples>360</samples>
+              <resolution>1</resolution>
+              <min_angle>0.0</min_angle>
+              <max_angle>6.28</max_angle>
+            </horizontal>
+          </scan>
+          <range>
+            <min>0.12</min>
+            <max>3.5</max>
+            <resolution>0.015</resolution>
+          </range>
+          <noise type="gaussian">
+            <mean>0.0</mean>
+            <stddev>0.01</stddev>
+          </noise>
+        </ray>
+        <plugin name="tb3_laser_ros" filename="libgazebo_ros_ray_sensor.so">
+          <ros>
+            <namespace>/</namespace>
+            <remapping>~/out:=scan</remapping>
+          </ros>
+          <output_type>sensor_msgs/LaserScan</output_type>
+          <frame_name>base_scan</frame_name>
+        </plugin>
+      </sensor>
+    </gazebo>
   <!-- RGB camera -->
-  <gazebo reference="oak_d_pro_color_optical_frame">
+  <gazebo reference="oak_d_pro_camera_gz">
     <sensor name="rgb_camera" type="camera">
-      <pose>0 0 0 3.14 -1.5708 1.5708</pose>
+          <pose>0 0 0 0 0 0</pose>
       <always_on>true</always_on>
       <update_rate>30</update_rate>
@@ -444,16 +446,18 @@
         <ros>
           <namespace>/</namespace>
-          <remapping>image_raw:=rgb_camera/image</remapping>
-          <remapping>camera_info:=rgb_camera/camera_info</remapping>
+          <!-- => /rgb_camera/image -->
+          <remapping>image_raw:=image</remapping>
+          <!-- => /rgb_camera/camera_info -->
+          <remapping>camera_info:=camera_info</remapping>
         </ros>
         <camera_name>rgb_camera</camera_name>
-        <frame_name>oak_d_pro_color_optical_frame</frame_name>
+            <frame_name>oak_d_pro_color_optical_frame</frame_name>
       </plugin>
     </sensor>
   </gazebo>
-  <!-- Depth camera (le même plugin peut sortir des images depth si le sensor est "depth") -->
+  <!-- Depth camera -->
   <gazebo reference="oak_d_pro_depth_optical_frame">
     <sensor name="depth_camera" type="depth">
-      <pose>0 0 0 0 0 0</pose>
+          <pose>0 0 0 0 0 0</pose>
       <always_on>true</always_on>
       <update_rate>30</update_rate>
@@ -464,4 +468,5 @@
           <width>640</width>
           <height>480</height>
+          <!-- tu peux laisser ça pour la partie "image", la profondeur sortira quand même en depth -->
           <format>R8G8B8</format>
         </image>
@@ -474,6 +479,8 @@
         <ros>
           <namespace>/</namespace>
-          <remapping>image_raw:=depth_camera/image</remapping>
-          <remapping>camera_info:=depth_camera/camera_info</remapping>
+          <!-- => /depth_camera/image -->
+          <remapping>image_raw:=image</remapping>
+          <!-- => /depth_camera/camera_info -->
+          <remapping>camera_info:=camera_info</remapping>
         </ros>
         <camera_name>depth_camera</camera_name>
@@ -505,17 +512,32 @@
     </plugin>
   </gazebo>
-  <!-- Joint states (remplace gz-sim-joint-state-publisher-system) -->
+  <!-- ros2_control: expose gripper joints -->
+  <ros2_control name="GazeboSystem" type="system">
+      <hardware>
+        <plugin>gazebo_ros2_control/GazeboSystem</plugin>
+      </hardware>
+      <joint name="gripper_left_joint">
+        <command_interface name="position"/>
+        <state_interface name="position"/>
+        <state_interface name="velocity"/>
+      </joint>
+      <joint name="gripper_right_joint">
+        <command_interface name="position"/>
+        <state_interface name="position"/>
+        <state_interface name="velocity"/>
+      </joint>
+      <joint name="wheel_left_joint">
+        <state_interface name="position"/>
+        <state_interface name="velocity"/>
+      </joint>
+      <joint name="wheel_right_joint">
+        <state_interface name="position"/>
+        <state_interface name="velocity"/>
+      </joint>
+    </ros2_control>
+  <!-- Gazebo ros2_control plugin -->
   <gazebo>
-    <plugin name="tb3_joint_state_pub" filename="libgazebo_ros_joint_state_publisher.so">
-      <ros>
-        <namespace>/</namespace>
-        <remapping>joint_states:=joint_states</remapping>
-      </ros>
-      <update_rate>30</update_rate>
-      <joint_name>wheel_left_joint</joint_name>
-      <joint_name>wheel_right_joint</joint_name>
-      <joint_name>gripper_tilt_joint</joint_name>
-      <joint_name>gripper_left_joint</joint_name>
-      <joint_name>gripper_right_joint</joint_name>
+    <plugin name="gazebo_ros2_control" filename="libgazebo_ros2_control.so">
+      <parameters>$(arg controllers_file)</parameters>
     </plugin>
   </gazebo>

Commit message: fix hitbox + gix patinage du turtle bot + approche manuelle ok + fix du controller

File: urdf/turtlebot3_burger_gripper.urdf.xacro (robot description, xacro)
@@ -261,13 +261,26 @@
     </visual>
     <collision>
-      <origin rpy="0 0 0" xyz="0.09 0 -0.02"/>
-      <geometry>
-        <box size="0.02 0.02 0.041"/>
-      </geometry>
-    </collision>
-    <inertial>
-        <origin xyz="0.045 0 -0.021"/>
-        <mass value="0.12000000"/>
-        <inertia ixx="23.07e-06" ixy="0.0" ixz="0.0" iyy="107.0e-06" iyz="0.0" izz="96.06e-06"/>
+      <origin rpy="0 0 0" xyz="0.095 0.01 -0.015"/>
+      <geometry>
+        <box size="0.015 0.015 0.04"/> </geometry>
+      <surface>
+        <friction>
+          <ode>
+            <mu>1000.0</mu>
+            <mu2>1000.0</mu2>
+          </ode>
+        </friction>
+        <contact>
+          <ode>
+            <kp>1000000.0</kp>
+            <kd>1.0</kd>
+            <min_depth>0.001</min_depth>
+          </ode>
+        </contact>
+      </surface>
+    </collision>
+    <inertial>
+      <origin xyz="0.045 0 -0.021"/>
+      <mass value="0.01"/> <inertia ixx="0.000001" ixy="0.0" ixz="0.0" iyy="0.000001" iyz="0.0" izz="0.000001"/>
     </inertial>
   </link>
@@ -288,13 +301,28 @@
     </visual>
     <collision>
-      <origin rpy="0 0 0" xyz="0.09 0 -0.02"/>
-      <geometry>
-        <box size="0.02 0.02 0.041"/>
-      </geometry>
-    </collision>
-    <inertial>
-        <origin xyz="0.045 0.0 -0.021"/>
-        <mass value="0.12000000"/>
-        <inertia ixx="23.20e-06" ixy="0.0" ixz="0.0" iyy="107.33e-06" iyz="0.0" izz="96.18e-06"/>
+      <origin rpy="0 0 0" xyz="0.095 -0.01 -0.015"/>
+      <geometry>
+        <box size="0.015 0.015 0.04"/>
+      </geometry>
+      <surface>
+        <friction>
+          <ode>
+            <mu>1000.0</mu>
+            <mu2>1000.0</mu2>
+          </ode>
+        </friction>
+        <contact>
+          <ode>
+            <kp>1000000.0</kp>
+            <kd>1.0</kd>
+            <min_depth>0.001</min_depth>
+          </ode>
+        </contact>
+      </surface>
+    </collision>
+    <inertial>
+      <origin xyz="0.045 0.0 -0.021"/>
+      <mass value="0.01"/>
+      <inertia ixx="0.000001" ixy="0.0" ixz="0.0" iyy="0.000001" iyz="0.0" izz="0.000001"/>
     </inertial>
   </link>
@@ -390,5 +418,4 @@
     </sensor>
   </gazebo>
-  <!-- LIDAR 2D (Gazebo Classic = ray/gpu_ray + <ray> ... ) -->
   <gazebo reference="base_scan">
       <sensor name="hls_lfcd_lds" type="ray">
@@ -424,5 +451,4 @@
       </sensor>
     </gazebo>
-  <!-- RGB camera -->
   <gazebo reference="oak_d_pro_camera_gz">
     <sensor name="rgb_camera" type="camera">
@@ -446,7 +472,5 @@
         <ros>
           <namespace>/</namespace>
-          <!-- => /rgb_camera/image -->
           <remapping>image_raw:=image</remapping>
-          <!-- => /rgb_camera/camera_info -->
           <remapping>camera_info:=camera_info</remapping>
         </ros>
@@ -456,5 +480,4 @@
     </sensor>
   </gazebo>
-  <!-- Depth camera -->
   <gazebo reference="oak_d_pro_depth_optical_frame">
     <sensor name="depth_camera" type="depth">
@@ -479,7 +502,5 @@
         <ros>
           <namespace>/</namespace>
-          <!-- => /depth_camera/image -->
           <remapping>image_raw:=image</remapping>
-          <!-- => /depth_camera/camera_info -->
           <remapping>camera_info:=camera_info</remapping>
         </ros>
@@ -489,5 +510,4 @@
     </sensor>
   </gazebo>
-  <!-- Diff drive (remplace gz-sim-diff-drive-system) -->
   <gazebo>
     <plugin name="tb3_diff_drive" filename="libgazebo_ros_diff_drive.so">
@@ -512,5 +532,4 @@
     </plugin>
   </gazebo>
-  <!-- ros2_control: expose gripper joints -->
   <ros2_control name="GazeboSystem" type="system">
       <hardware>
@@ -536,5 +555,4 @@
       </joint>
     </ros2_control>
-  <!-- Gazebo ros2_control plugin -->
   <gazebo>
     <plugin name="gazebo_ros2_control" filename="libgazebo_ros2_control.so">
@@ -542,3 +560,12 @@
     </plugin>
   </gazebo>
+  <gazebo reference="caster_back_link">
+    <mu1>0.0</mu1>
+    <mu2>0.0</mu2>
+    <kp>1000000.0</kp>
+    <kd>100.0</kd>
+    <minDepth>0.001</minDepth>
+    <maxVel>1.0</maxVel>
+    <material>Gazebo/Grey</material>
+  </gazebo>
 </robot>

Commit message: robot plus fluide + plus rapide + plus classe + fix return home

File: urdf/turtlebot3_burger_gripper.urdf.xacro (robot description, xacro)
@@ -338,7 +338,7 @@
       <origin xyz="0.0 0.0 0.0" rpy="0 0 0"/>
       <geometry>
-          <mesh filename="package://tb3_autonomy/meshes/sensors/OAK-D-PRO.stl" scale="1.0 1.0 1.0"/>
-      </geometry>
-      <material name="dark"/>
+          <mesh filename="package://tb3_autonomy/meshes/sensors/OAK-D-PRO.dae" scale="1.0 1.0 1.0"/>
+      </geometry>
+      <material name="grey"/>
     </visual>
     <inertial>
@@ -456,5 +456,5 @@
       <always_on>true</always_on>
       <update_rate>30</update_rate>
-      <visualize>true</visualize>
+      <visualize>false</visualize>
       <camera>
         <horizontal_fov>1.047</horizontal_fov>
@@ -485,5 +485,5 @@
       <always_on>true</always_on>
       <update_rate>30</update_rate>
-      <visualize>true</visualize>
+      <visualize>false</visualize>
       <camera>
         <horizontal_fov>1.047</horizontal_fov>
